Commit message: Add jolo (Jenna's Only Look Once) buoy detection model.

File: urdf/izzyboat.urdf (robot description, URDF)
Before this commit: robot izzyboat, 5 links, 4 joints
Links:
- removed link izzy/sensors/cameras/oak_rgb_camera_optical_frame
- added link izzy/forward_oak_camera_optical_frame
Joints:
- joint forward_optical_to_oak_optical: child izzy/sensors/cameras/oak_rgb_camera_optical_frame -> izzy/forward_oak_camera_optical_frame

Commit message: Update tf and launch for jolo

File: urdf/izzyboat.urdf (robot description, URDF)
Before this commit: robot izzyboat, 5 links, 4 joints
Links:
- removed link izzy/forward_oak_camera_optical_frame
- added link forward_oak_rgb_camera_optical_frame
Joints:
- joint forward_optical_to_oak_optical: child izzy/forward_oak_camera_optical_frame -> forward_oak_rgb_camera_optical_frame

Commit message: Update urdf with correct oak camera frame

File: urdf/izzyboat.urdf (robot description, URDF)
Before this commit: robot izzyboat, 5 links, 4 joints
Links:
- removed link forward_oak_rgb_camera_optical_frame
- added link izzy/forward_oak_camera; visual cylinder length=0.07 radius=0.05
- added link izzy/forward_oak_camera_optical_frame
Joints:
- added joint base_to_oak_forward: type fixed, parent izzy/base_link, child izzy/forward_oak_camera, origin xyz=0 0 0.5 rpy=0 0 0
- added joint oak_forward_to_oak_forward_optical: type fixed, parent izzy/forward_oak_camera, child izzy/forward_oak_camera_optical_frame, origin xyz=0 0 0 rpy=-1.57075 0 -1.57075
- joint forward_optical_to_oak_optical: child forward_oak_rgb_camera_optical_frame -> izzy/forward_oak_camera_optical_frame

Commit message: Add norbit driver with basic soundings output

File: urdf/izzyboat.urdf (robot description, URDF)
Before this commit: robot izzyboat, 6 links, 6 joints
Links:
- added link izzy/norbit; visual box size=0.15 0.15 0.1
Joints:
- added joint base_to_norbit: type fixed, parent izzy/base_link, child izzy/norbit, origin xyz=0 0 -0.18 rpy=3.14159 0.0 0.0

Commit message: Update urdf

File: urdf/izzyboat.urdf (robot description, URDF)
Before this commit: robot izzyboat, 7 links, 7 joints
Links:
- removed link izzy/norbit
Joints:
- removed joint base_to_norbit
- joint base_to_camera_forward: origin xyz=1.55 0 -0.055 rpy=0 0 0 -> xyz=1.55 0 0.5 rpy=0 0 0
- joint base_to_deltat: origin xyz=0 0 -0.65 rpy=3.14159 0 3.14159 -> xyz=0 0 -0.15 rpy=3.14159 0 3.14159
- joint base_to_oak_forward: origin xyz=0 0 0.5 rpy=0 0 0 -> xyz=-0.1 0 1.0 rpy=0 0 0

Commit message: Update urdf

File: urdf/izzyboat.urdf (robot description, URDF)
Before this commit: robot izzyboat, 6 links, 6 joints
Joints:
- joint base_to_camera_forward: origin xyz=1.55 0 0.5 rpy=0 0 0 -> xyz=1.25 0 0.5 rpy=0 0 0
- joint base_to_deltat: origin xyz=0 0 -0.15 rpy=3.14159 0 3.14159 -> xyz=-.1530 0 -0.15 rpy=3.14159 0 3.14159
- joint base_to_oak_forward: origin xyz=-0.1 0 1.0 rpy=0 0 0 -> xyz=0.378 0 1.241 rpy=0 0 0

Commit message: Add top camera

File: urdf/izzyboat.urdf (robot description, URDF)
Before this commit: robot izzyboat, 6 links, 6 joints
Links:
- removed link izzy/forward_oak_camera_optical_frame
- added link izzy/forward_oak_camera_optical
- added link izzy/top_camera; visual cylinder length=0.07 radius=0.05
- added link izzy/top_camera_optical
Joints:
- removed joint forward_optical_to_oak_optical
- added joint oak_to_top: type fixed, parent izzy/forward_oak_camera, child izzy/top_camera, origin xyz=0 0 0.28 rpy=0 1.0 0
- added joint top_to_top_optical: type fixed, parent izzy/top_camera, child izzy/top_camera_optical, origin xyz=0 0 0 rpy=-1.57075 0 -1.57075
- joint base_to_oak_forward: origin xyz=0.378 0 1.241 rpy=0 0 0 -> xyz=0.378 0 1.241 rpy=0 -0.04 0
- joint oak_forward_to_oak_forward_optical: child izzy/forward_oak_camera_optical_frame -> izzy/forward_oak_camera_optical

Commit message: Update cameras

File: urdf/izzyboat.urdf (robot description, URDF)
Before this commit: robot izzyboat, 8 links, 7 joints
Joints:
- joint base_to_oak_forward: origin xyz=0.378 0 1.241 rpy=0 -0.04 0 -> xyz=0.378 0 1.241 rpy=-0.01 0.04 0
