Commit message: fix: address review feedback on URDF and configs (#25)
- Rename USB camera frames to bizzy/usb_camera to match perception_launch.py
- Fix hull mesh z-origin: deck at z=0, bottom at z=-0.3 (matches base_link)
- Correct bizzyboat.yaml width to 0.9m and color to yellow
- Update package creation doc to reference .urdf.xacro

File: bizzyboat_project11/urdf/bizzyboat.urdf.xacro (robot description, xacro)
@@ -87,5 +87,5 @@
   <!-- ========== Factory USB Camera ========== -->
   <!-- On the crossbar rail, toward the bow. -->
-  <link name="bizzy/camera_usb">
+  <link name="bizzy/usb_camera">
     <visual>
       <geometry>
@@ -96,13 +96,13 @@
     </visual>
   </link>
-  <joint name="base_to_camera_usb" type="fixed">
+  <joint name="base_to_usb_camera" type="fixed">
     <parent link="bizzy/base_link"/>
-    <child link="bizzy/camera_usb"/>
+    <child link="bizzy/usb_camera"/>
     <origin xyz="0.55 0.0 1.15" rpy="0 0 0"/>
   </joint>
-  <link name="bizzy/camera_usb_optical"/>
-  <joint name="camera_usb_to_camera_usb_optical" type="fixed">
-    <parent link="bizzy/camera_usb"/>
-    <child link="bizzy/camera_usb_optical"/>
+  <link name="bizzy/usb_camera_optical"/>
+  <joint name="usb_camera_to_usb_camera_optical" type="fixed">
+    <parent link="bizzy/usb_camera"/>
+    <child link="bizzy/usb_camera_optical"/>
     <origin xyz="0 0 0" rpy="${-pi/2} 0 ${-pi/2}"/>
   </joint>

Commit message: bizzyboat URDF: measured waterline frame + sidescan offsets (#282)
2026-06-15 Lake Massabesic measured values:
- Add bizzy/waterline frame at +0.030 m above base_link (draft ref +0.180 m,
  water 0.150 m below ref). Supports datum / sea-surface reference (#278).
- Correct garmin_sidescan mount: x 0.15->-0.003, z -0.30->-0.29 (essentially
  centered, was approximate).

Verified: xacro expands, check_urdf parses, origins correct. The hand-maintained
docs/bizzyboat_offsets.svg is decoupled from the URDF and omits sidescan/
waterline — diagram update deferred (separate doc task).

Closes #282

File: bizzyboat_project11/urdf/bizzyboat.urdf.xacro (robot description, xacro)
@@ -117,4 +117,14 @@
     </visual>
   </link>
+  <!-- ========== Reference frames ========== -->
+  <!-- Measured water surface, 2026-06-15 Lake Massabesic: draft reference point
+       +0.180 m above base_link, waterline 0.150 m below that ref => waterline
+       +0.030 m above base_link (base_link sits ~30 mm below the surface). -->
+  <link name="bizzy/waterline"/>
+  <joint name="base_to_waterline" type="fixed">
+    <parent link="bizzy/base_link"/>
+    <child link="bizzy/waterline"/>
+    <origin xyz="0 0 0.030" rpy="0 0 0"/>
+  </joint>
   <!-- ========== Cameras (4x OAK-1 PoE) ========== -->
   <!-- Mounted at top of mast on 3D-printed bracket, 90deg apart.
@@ -207,13 +217,13 @@
     x="-0.23" y="0.0" z="-0.145"/>
   <!-- ========== Garmin GCV-20 Sidescan ========== -->
-  <!-- Centered, ~0.15 m forward of base_link, flush against the hull underside.
-       z = -0.30 is the flat hull bottom (hull depth 0.30 below the deck/base_link
+  <!-- Measured 2026-06-15 (Lake Massabesic): essentially centered (3 mm aft of
+       base_link), against the hull underside. z = -0.29 is the transducer face,
+       just above the flat hull bottom (hull depth ~0.30 below the deck/base_link
        plane per scripts/generate_hull_mesh.py). The garmin_sidescan driver stamps
        each channel image with a per-channel frame_id — the base frame_id param
        ("bizzy/garmin_sidescan", set in launch/sidescan_launch.py) plus a channel
        suffix, giving "bizzy/garmin_sidescan_down/_port/_starboard"; this macro
-       supplies the matching TF frames.
-       Offsets are approximate — confirm by measurement. -->
+       supplies the matching TF frames. -->
   <xacro:garmin_sidescan parent="bizzy/base_link" name="garmin_sidescan"
-    x="0.15" y="0.0" z="-0.30"/>
+    x="-0.003" y="0.0" z="-0.29"/>
 </robot>
