Commit message: fix: replace lateral crossbar with fore-aft center rail in URDF (#25)
The actual boat has a fore-aft center rail along y=0, not a lateral
crossbar. Updated mast geometry, moved USB camera to rail height
(z=0.89), and updated sensor positions from rough measurements.

Co-Authored-By: Claude Opus 4.6 (1M context) <noreply@anthropic.com>

File: bizzyboat_project11/urdf/bizzyboat.urdf.xacro (robot description, xacro)
@@ -35,25 +35,29 @@
       <material name="bumper_black"/>
     </visual>
-    <!-- Mast uprights (two vertical stainless steel tubes) -->
+    <!-- Mast uprights (two vertical stainless steel tubes).
+         Port upright extends to camera bracket at top (~z=1.41).
+         Starboard upright extends to center rail height (~z=0.89). -->
     <visual name="mast_port">
       <geometry>
-        <box size="0.04 0.04 0.95"/>
+        <box size="0.04 0.04 1.11"/>
       </geometry>
-      <origin xyz="0.15 0.35 0.775"/>
+      <origin xyz="0.15 0.35 0.855"/>
       <material name="metal_gray"/>
     </visual>
     <visual name="mast_starboard">
       <geometry>
-        <box size="0.04 0.04 0.95"/>
+        <box size="0.04 0.04 0.59"/>
       </geometry>
-      <origin xyz="0.15 -0.35 0.775"/>
+      <origin xyz="0.15 -0.35 0.595"/>
       <material name="metal_gray"/>
     </visual>
-    <!-- Horizontal crossbar connecting mast uprights -->
-    <visual name="crossbar">
+    <!-- Fore-aft center rail along y=0, supported by the two uprights.
+         GNSS antennas mount at the forward and aft ends; USB camera
+         and other equipment mount between them. -->
+    <visual name="center_rail">
       <geometry>
-        <box size="0.04 0.80 0.04"/>
+        <box size="1.67 0.04 0.04"/>
       </geometry>
-      <origin xyz="0.15 0.0 1.15"/>
+      <origin xyz="0.0 0.0 0.89"/>
       <material name="metal_gray"/>
     </visual>
@@ -63,6 +67,6 @@
        All tilted ~10deg downward (pitch = -0.17 rad).
        Positions are estimated [EST] — refine with measurements. -->
-  <xacro:property name="cam_x" value="0.15"/>
-  <xacro:property name="cam_z" value="1.25"/>
+  <xacro:property name="cam_x" value="0.31"/>
+  <xacro:property name="cam_z" value="1.41"/>
   <xacro:property name="cam_tilt" value="-0.17"/>
   <xacro:oak_camera parent="bizzy/base_link" name="oak_forward"
@@ -79,10 +83,10 @@
     pitch="${cam_tilt}" yaw="${pi}"/>
   <!-- ========== GNSS Antennas (2x CUAV C-RTK 2HP) ========== -->
-  <!-- Black pucks in white brackets on crossbar ends.
-       Baseline ~0.80m. Positions are estimated [EST]. -->
-  <xacro:gnss_antenna parent="bizzy/base_link" name="gnss_port"
-    x="0.15" y="0.40" z="1.15"/>
-  <xacro:gnss_antenna parent="bizzy/base_link" name="gnss_starboard"
-    x="0.15" y="-0.40" z="1.15"/>
+  <!-- Black pucks fore and aft. Baseline ~1.67m.
+       Measured from base_link (center screw hole). -->
+  <xacro:gnss_antenna parent="bizzy/base_link" name="gnss_forward"
+    x="0.835" y="0.0" z="0.89"/>
+  <xacro:gnss_antenna parent="bizzy/base_link" name="gnss_aft"
+    x="-0.835" y="0.0" z="0.89"/>
   <!-- ========== Factory USB Camera ========== -->
   <!-- On the crossbar rail, toward the bow. -->
@@ -99,5 +103,5 @@
     <parent link="bizzy/base_link"/>
     <child link="bizzy/usb_camera"/>
-    <origin xyz="0.55 0.0 1.15" rpy="0 0 0"/>
+    <origin xyz="0.55 0.0 0.89" rpy="0 0 0"/>
   </joint>
   <link name="bizzy/usb_camera_optical"/>
@@ -107,8 +111,33 @@
     <origin xyz="0 0 0" rpy="${-pi/2} 0 ${-pi/2}"/>
   </joint>
+  <!-- ========== AutoNav Box (contains Cube Orange FCU + IMU) ========== -->
+  <!-- Front bottom of box at (-0.875, 0, -0.01) from base_link.
+       Box dimensions ~0.20 x 0.15 x 0.15 estimated from photos.
+       IMU is inside the Cube Orange, position within box is approximate. -->
+  <link name="bizzy/autonav_box">
+    <visual>
+      <geometry>
+        <box size="0.20 0.15 0.15"/>
+      </geometry>
+      <origin xyz="-0.10 0 0.075"/>
+      <material name="bumper_black"/>
+    </visual>
+  </link>
+  <joint name="base_to_autonav_box" type="fixed">
+    <parent link="bizzy/base_link"/>
+    <child link="bizzy/autonav_box"/>
+    <origin xyz="-0.875 0.0 -0.01" rpy="0 0 0"/>
+  </joint>
+  <!-- IMU frame at estimated center of Cube Orange inside the box -->
+  <link name="bizzy/imu"/>
+  <joint name="autonav_box_to_imu" type="fixed">
+    <parent link="bizzy/autonav_box"/>
+    <child link="bizzy/imu"/>
+    <origin xyz="-0.10 0.0 0.075" rpy="0 0 0"/>
+  </joint>
   <!-- ========== Imagenex DeltaT Sonar ========== -->
   <!-- Below hull, approximate position from manual diagram.
        Exact mount position TBD. -->
   <xacro:deltat_sonar parent="bizzy/base_link" name="deltat"
-    x="-0.15" y="0.0" z="-0.15"/>
+    x="-0.23" y="0.0" z="-0.18"/>
 </robot>

Commit message: feat: flesh out mast frame geometry and add hull gunwales (#25)
Replace simplified two-upright mast with rectangular cage frame
matching photos: four uprights, lateral crossbars, fore-aft side
rails, risers, and camera mast extension. Regenerate hull mesh
with gunwale walls (0.25m amidships, 0.35m bow rake) and bathtub
interior visible from above.

Co-Authored-By: Claude Opus 4.6 (1M context) <noreply@anthropic.com>

File: bizzyboat_project11/urdf/bizzyboat.urdf.xacro (robot description, xacro)
@@ -35,29 +35,78 @@
       <material name="bumper_black"/>
     </visual>
-    <!-- Mast uprights (two vertical stainless steel tubes).
-         Port upright extends to camera bracket at top (~z=1.41).
-         Starboard upright extends to center rail height (~z=0.89). -->
-    <visual name="mast_port">
-      <geometry>
-        <box size="0.04 0.04 1.11"/>
-      </geometry>
-      <origin xyz="0.15 0.35 0.855"/>
+    <!-- ── Mast frame ──
+         Rectangular cage visible in photos: four uprights at hull
+         corners, lateral crossbars fore and aft, fore-aft side rails,
+         risers to center rail, and a camera mast extension.
+         Uprights rise from hull gunwale (~z=0.30) to crossbar
+         height (z=0.77, from measurement sketch). -->
+    <!-- Four uprights (hull gunwale to crossbar height) -->
+    <visual name="mast_fwd_port">
+      <geometry><box size="0.04 0.04 0.47"/></geometry>
+      <origin xyz="0.30 0.35 0.535"/>
       <material name="metal_gray"/>
     </visual>
-    <visual name="mast_starboard">
-      <geometry>
-        <box size="0.04 0.04 0.59"/>
-      </geometry>
-      <origin xyz="0.15 -0.35 0.595"/>
+    <visual name="mast_fwd_stbd">
+      <geometry><box size="0.04 0.04 0.47"/></geometry>
+      <origin xyz="0.30 -0.35 0.535"/>
       <material name="metal_gray"/>
     </visual>
-    <!-- Fore-aft center rail along y=0, supported by the two uprights.
+    <visual name="mast_aft_port">
+      <geometry><box size="0.04 0.04 0.47"/></geometry>
+      <origin xyz="-0.40 0.35 0.535"/>
+      <material name="metal_gray"/>
+    </visual>
+    <visual name="mast_aft_stbd">
+      <geometry><box size="0.04 0.04 0.47"/></geometry>
+      <origin xyz="-0.40 -0.35 0.535"/>
+      <material name="metal_gray"/>
+    </visual>
+    <!-- Lateral crossbars (port-to-starboard at top of uprights) -->
+    <visual name="crossbar_fwd">
+      <geometry><box size="0.04 0.70 0.04"/></geometry>
+      <origin xyz="0.30 0.0 0.77"/>
+      <material name="metal_gray"/>
+    </visual>
+    <visual name="crossbar_aft">
+      <geometry><box size="0.04 0.70 0.04"/></geometry>
+      <origin xyz="-0.40 0.0 0.77"/>
+      <material name="metal_gray"/>
+    </visual>
+    <!-- Fore-aft side rails (connecting forward and aft bents) -->
+    <visual name="rail_port">
+      <geometry><box size="0.70 0.04 0.04"/></geometry>
+      <origin xyz="-0.05 0.35 0.77"/>
+      <material name="metal_gray"/>
+    </visual>
+    <visual name="rail_stbd">
+      <geometry><box size="0.70 0.04 0.04"/></geometry>
+      <origin xyz="-0.05 -0.35 0.77"/>
+      <material name="metal_gray"/>
+    </visual>
+    <!-- Risers from crossbars to center rail height -->
+    <visual name="riser_fwd">
+      <geometry><box size="0.04 0.04 0.12"/></geometry>
+      <origin xyz="0.30 0.0 0.83"/>
+      <material name="metal_gray"/>
+    </visual>
+    <visual name="riser_aft">
+      <geometry><box size="0.04 0.04 0.12"/></geometry>
+      <origin xyz="-0.40 0.0 0.83"/>
+      <material name="metal_gray"/>
+    </visual>
+    <!-- Fore-aft center rail along y=0 (z=0.89).
          GNSS antennas mount at the forward and aft ends; USB camera
-         and other equipment mount between them. -->
+         and other equipment mount between them. Overhangs the frame
+         to reach the GNSS positions at x=±0.835. -->
     <visual name="center_rail">
-      <geometry>
-        <box size="1.67 0.04 0.04"/>
-      </geometry>
+      <geometry><box size="1.67 0.04 0.04"/></geometry>
       <origin xyz="0.0 0.0 0.89"/>
+      <material name="metal_gray"/>
+    </visual>
+    <!-- Camera mast (vertical extension above forward-port upright
+         to camera bracket at z=1.41) -->
+    <visual name="camera_mast">
+      <geometry><box size="0.04 0.04 0.64"/></geometry>
+      <origin xyz="0.31 0.35 1.09"/>
       <material name="metal_gray"/>
     </visual>

Commit message: fix: slanted uprights, hull normals, camera tilt, and rail/camera positions (#25)
- Fix hull mesh normals (face winding was inverted) and add double-sided
  end caps so stern is visible from interior
- Slant mast uprights inward (~23 deg) matching photos and front view diagram
- Move camera tower to centerline (factory WiFi mast extended for OAK cameras)
- Extend center rail to 2.1m matching top view diagram (well past GNSS antennas)
- Move USB camera to rail end (x=1.05), forward of GNSS antennas
- Fix OAK camera tilt to 5 deg downward (pitch sign was inverted)

Co-Authored-By: Claude Opus 4.6 (1M context) <noreply@anthropic.com>

File: bizzyboat_project11/urdf/bizzyboat.urdf.xacro (robot description, xacro)
@@ -36,38 +36,41 @@
     </visual>
     <!-- ── Mast frame ──
-         Rectangular cage visible in photos: four uprights at hull
-         corners, lateral crossbars fore and aft, fore-aft side rails,
-         risers to center rail, and a camera mast extension.
+         A-frame cage visible in photos: four slanted uprights lean
+         inward from hull sides (y≈±0.38) to frame top (y≈±0.18),
+         lateral crossbars fore and aft, fore-aft side rails, risers
+         to center rail, and the factory WiFi tower extended for cameras.
          Uprights rise from hull gunwale (~z=0.30) to crossbar
-         height (z=0.77, from measurement sketch). -->
-    <!-- Four uprights (hull gunwale to crossbar height) -->
+         height (z=0.77, from measurement sketch).
+         Roll angle: atan2(0.20, 0.47) ≈ 0.40 rad (~23 deg). -->
+    <!-- Four slanted uprights (hull gunwale to crossbar height).
+         Lean inward: bottom at y≈±0.38, top at y≈±0.18. -->
     <visual name="mast_fwd_port">
-      <geometry><box size="0.04 0.04 0.47"/></geometry>
-      <origin xyz="0.30 0.35 0.535"/>
+      <geometry><box size="0.04 0.04 0.51"/></geometry>
+      <origin xyz="0.30 0.28 0.535" rpy="0.40 0 0"/>
       <material name="metal_gray"/>
     </visual>
     <visual name="mast_fwd_stbd">
-      <geometry><box size="0.04 0.04 0.47"/></geometry>
-      <origin xyz="0.30 -0.35 0.535"/>
+      <geometry><box size="0.04 0.04 0.51"/></geometry>
+      <origin xyz="0.30 -0.28 0.535" rpy="-0.40 0 0"/>
       <material name="metal_gray"/>
     </visual>
     <visual name="mast_aft_port">
-      <geometry><box size="0.04 0.04 0.47"/></geometry>
-      <origin xyz="-0.40 0.35 0.535"/>
+      <geometry><box size="0.04 0.04 0.51"/></geometry>
+      <origin xyz="-0.40 0.28 0.535" rpy="0.40 0 0"/>
       <material name="metal_gray"/>
     </visual>
     <visual name="mast_aft_stbd">
-      <geometry><box size="0.04 0.04 0.47"/></geometry>
-      <origin xyz="-0.40 -0.35 0.535"/>
+      <geometry><box size="0.04 0.04 0.51"/></geometry>
+      <origin xyz="-0.40 -0.28 0.535" rpy="-0.40 0 0"/>
       <material name="metal_gray"/>
     </visual>
     <!-- Lateral crossbars (port-to-starboard at top of uprights) -->
     <visual name="crossbar_fwd">
-      <geometry><box size="0.04 0.70 0.04"/></geometry>
+      <geometry><box size="0.04 0.36 0.04"/></geometry>
       <origin xyz="0.30 0.0 0.77"/>
       <material name="metal_gray"/>
     </visual>
     <visual name="crossbar_aft">
-      <geometry><box size="0.04 0.70 0.04"/></geometry>
+      <geometry><box size="0.04 0.36 0.04"/></geometry>
       <origin xyz="-0.40 0.0 0.77"/>
       <material name="metal_gray"/>
@@ -76,10 +79,10 @@
     <visual name="rail_port">
       <geometry><box size="0.70 0.04 0.04"/></geometry>
-      <origin xyz="-0.05 0.35 0.77"/>
+      <origin xyz="-0.05 0.18 0.77"/>
       <material name="metal_gray"/>
     </visual>
     <visual name="rail_stbd">
       <geometry><box size="0.70 0.04 0.04"/></geometry>
-      <origin xyz="-0.05 -0.35 0.77"/>
+      <origin xyz="-0.05 -0.18 0.77"/>
       <material name="metal_gray"/>
     </visual>
@@ -96,17 +99,18 @@
     </visual>
     <!-- Fore-aft center rail along y=0 (z=0.89).
-         GNSS antennas mount at the forward and aft ends; USB camera
-         and other equipment mount between them. Overhangs the frame
-         to reach the GNSS positions at x=±0.835. -->
+         Runs nearly the full length of the boat (top view diagram,
+         Fig 139). GNSS antennas and USB camera mount along it;
+         the rail extends well past the antennas on both ends. -->
     <visual name="center_rail">
-      <geometry><box size="1.67 0.04 0.04"/></geometry>
+      <geometry><box size="2.10 0.04 0.04"/></geometry>
       <origin xyz="0.0 0.0 0.89"/>
       <material name="metal_gray"/>
     </visual>
-    <!-- Camera mast (vertical extension above forward-port upright
-         to camera bracket at z=1.41) -->
-    <visual name="camera_mast">
-      <geometry><box size="0.04 0.04 0.64"/></geometry>
-      <origin xyz="0.31 0.35 1.09"/>
+    <!-- Factory WiFi tower, extended for 4x OAK camera bracket.
+         Single vertical tube on centerline, rising from center rail
+         to camera bracket height. -->
+    <visual name="camera_tower">
+      <geometry><box size="0.04 0.04 0.52"/></geometry>
+      <origin xyz="0.31 0.0 1.15"/>
       <material name="metal_gray"/>
     </visual>
@@ -114,9 +118,9 @@
   <!-- ========== Cameras (4x OAK-1 PoE) ========== -->
   <!-- Mounted at top of mast on 3D-printed bracket, 90deg apart.
-       All tilted ~10deg downward (pitch = -0.17 rad).
+       All tilted ~5deg downward (pitch = +0.09 rad in URDF convention).
        Positions are estimated [EST] — refine with measurements. -->
   <xacro:property name="cam_x" value="0.31"/>
   <xacro:property name="cam_z" value="1.41"/>
-  <xacro:property name="cam_tilt" value="-0.17"/>
+  <xacro:property name="cam_tilt" value="0.09"/>
   <xacro:oak_camera parent="bizzy/base_link" name="oak_forward"
     x="${cam_x}" y="0" z="${cam_z}"
@@ -139,5 +143,5 @@
     x="-0.835" y="0.0" z="0.89"/>
   <!-- ========== Factory USB Camera ========== -->
-  <!-- On the crossbar rail, toward the bow. -->
+  <!-- On the center rail, forward of the bow GNSS antenna. -->
   <link name="bizzy/usb_camera">
     <visual>
@@ -152,5 +156,5 @@
     <parent link="bizzy/base_link"/>
     <child link="bizzy/usb_camera"/>
-    <origin xyz="0.55 0.0 0.89" rpy="0 0 0"/>
+    <origin xyz="1.05 0.0 0.89" rpy="0 0 0"/>
   </joint>
   <link name="bizzy/usb_camera_optical"/>

Commit message: fix: refine AutoNav box dimensions and IMU position, add FCU custom params
Updated AutoNav box and IMU measurements from IzzyBoat photos (same model):
- Box: 0.23 x 0.28 x 0.14m (was 0.20 x 0.15 x 0.15 estimated)
- IMU at (-0.99, 0.0, 0.05) from base_link (was -0.975, 0.0, 0.065)

Added bizzyboat_fcu_custom.param as overlay tracking all FCU customizations
(GPS offsets, moving baseline, IMU position). INS_POS1/2/3 applied to FCU
via mavproxy on 2026-04-07.

Closes #37

Co-Authored-By: Claude Opus 4.6 (1M context) <noreply@anthropic.com>

File: bizzyboat_project11/urdf/bizzyboat.urdf.xacro (robot description, xacro)
@@ -166,12 +166,13 @@
   <!-- ========== AutoNav Box (contains Cube Orange FCU + IMU) ========== -->
   <!-- Front bottom of box at (-0.875, 0, -0.01) from base_link.
-       Box dimensions ~0.20 x 0.15 x 0.15 estimated from photos.
-       IMU is inside the Cube Orange, position within box is approximate. -->
+       Box dimensions 0.23 x 0.28 x 0.14 measured from IzzyBoat AutoNav photos
+       (same model used on BizzyBoat). X=depth(fore-aft), Y=width, Z=height.
+       IMU is inside the Cube Orange in the lower compartment. -->
   <link name="bizzy/autonav_box">
     <visual>
       <geometry>
-        <box size="0.20 0.15 0.15"/>
+        <box size="0.23 0.28 0.14"/>
       </geometry>
-      <origin xyz="-0.10 0 0.075"/>
+      <origin xyz="-0.115 0 0.07"/>
       <material name="bumper_black"/>
     </visual>
@@ -182,10 +183,12 @@
     <origin xyz="-0.875 0.0 -0.01" rpy="0 0 0"/>
   </joint>
-  <!-- IMU frame at estimated center of Cube Orange inside the box -->
+  <!-- IMU frame at Cube Orange center in the lower compartment.
+       Position from IzzyBoat AutoNav measurement photos (2024-06-14):
+       ~0.115m aft of box front, centered laterally, ~0.06m above box bottom. -->
   <link name="bizzy/imu"/>
   <joint name="autonav_box_to_imu" type="fixed">
     <parent link="bizzy/autonav_box"/>
     <child link="bizzy/imu"/>
-    <origin xyz="-0.10 0.0 0.075" rpy="0 0 0"/>
+    <origin xyz="-0.115 0.0 0.06" rpy="0 0 0"/>
   </joint>
   <!-- ========== Imagenex DeltaT Sonar ========== -->

Commit message: bizzyboat URDF: add M3 multibeam transducer frame (base_link -> m3)
cube_bathymetry georeferences soundings via a TF lookup to the map frame,
so the M3 needs a frame in the tree. Adds an m3_multibeam xacro macro and
instantiates bizzy/m3 at the #77 install offsets (x=-0.23 shared DeltaT
cavity, z=-0.145 transducer face, [MEAS] rough) with rpy=(pi,0,0) -- roll
pi maps base_link {x-fwd,y-port,z-up} to the sonar frame {x-fwd,y-stbd,
z-down}, matching the Kongsberg "normally mounted looking down" convention
and the SonarDetections frame kongsberg_em_bridge produces.

kongsberg_em_bridge must stamp frame_id "bizzy/m3" (launch param). Offsets
and orientation to be confirmed by a patch test.

Validated: full bizzyboat.urdf.xacro processes; base_to_m3 joint resolves to
rpy="3.14159 0 0" xyz="-0.23 0.0 -0.145".

Closes #221. Part of #77.

Co-Authored-By: Claude Opus 4.8 (1M context) <noreply@anthropic.com>

File: bizzyboat_project11/urdf/bizzyboat.urdf.xacro (robot description, xacro)
@@ -197,3 +197,11 @@
   <xacro:deltat_sonar parent="bizzy/base_link" name="deltat"
     x="-0.23" y="0.0" z="-0.18"/>
+  <!-- ========== Kongsberg M3 Multibeam ========== -->
+  <!-- Loaner unit sharing the DeltaT cavity (x); transducer-face z from the
+       #77 install log ([MEAS] rough). Frame consumed by cube_bathymetry's
+       TF lookup; kongsberg_em_bridge must stamp frame_id "bizzy/m3" (set its
+       frame_id param in the launch). Offsets + orientation to be confirmed by
+       a patch test. -->
+  <xacro:m3_multibeam parent="bizzy/base_link" name="m3"
+    x="-0.23" y="0.0" z="-0.145"/>
 </robot>

File: bizzyboat_project11/urdf/sensors/sonar.xacro (robot description, xacro)
@@ -20,3 +20,27 @@
     </joint>
   </xacro:macro>
+  <!-- Kongsberg M3 multibeam sonar macro.
+       Normally mounted below the hull looking down: roll=pi maps base_link
+       {x-fwd, y-port, z-up} to the sonar frame {x-fwd, y-starboard, z-down},
+       matching the Kongsberg "normally mounted looking down" convention
+       (EM Datagram Formats 850-160692 Note 1) and the
+       marine_acoustic_msgs/SonarDetections frame produced by kongsberg_em_bridge.
+       No yaw (unlike the DeltaT). Orientation is the nominal convention; a
+       patch test confirms/refines it (and resolves handedness). -->
+  <xacro:macro name="m3_multibeam" params="parent name x y z roll:=3.14159 yaw:=0">
+    <link name="bizzy/${name}">
+      <visual>
+        <geometry>
+          <box size="0.12 0.10 0.08"/>
+        </geometry>
+        <origin xyz="0 0 0"/>
+        <material name="sonar_gray"/>
+      </visual>
+    </link>
+    <joint name="base_to_${name}" type="fixed">
+      <parent link="${parent}"/>
+      <child link="bizzy/${name}"/>
+      <origin xyz="${x} ${y} ${z}" rpy="${roll} 0 ${yaw}"/>
+    </joint>
+  </xacro:macro>
 </robot>
