Commit message: fix(urdf): pitch camera mast -1.85 deg bow-up; reparent OAK cameras
Field change (2026-07-20): a new mast brace left the 4-camera bracket pitched bow-up, so the forward camera projected the far shoreline as obstacles ~35 m ahead. Adds a bizzy/camera_mast link rotated -1.85 deg about base_link Y and reparents all four OAK cameras (forward/port/starboard/aft) to it so they rotate rigidly together. Roll component still unmeasured (refine after on-water test). Committed as-is from the field working tree; not rebuilt/tested here. See docs/logs/2026/2026-07-20_gabby_logs.md.

Co-Authored-By: Claude Opus 4.8 (1M context) <noreply@anthropic.com>

File: bizzyboat_project11/urdf/bizzyboat.urdf.xacro (robot description, xacro)
@@ -134,15 +134,36 @@
   <xacro:property name="cam_z" value="1.41"/>
   <xacro:property name="cam_tilt" value="0.09"/>
-  <xacro:oak_camera parent="bizzy/base_link" name="oak_forward"
-    x="${cam_x}" y="0" z="${cam_z}"
+  <!-- Camera-mast remount correction (2026-07-20): a new mast brace left the
+       whole 4-camera bracket pitched slightly bow-up, so the forward camera
+       projected the far shoreline as obstacles ~35 m ahead. Estimated in the
+       field from forward-vs-aft segmentation horizons compared to TF: a rigid
+       mast pitch of ~1.85 deg (forward axis measured +2.32 deg up, aft -1.38
+       deg down; opposite-signed => antisymmetric (fwd-aft)/2 = 1.85 deg).
+       Modeled as ONE rotation of a common mast frame about base_link Y
+       (bow-up = negative URDF pitch, opposite the +0.09 down-tilt), so all
+       four cameras rotate rigidly together. A per-camera cam_tilt change would
+       be wrong: it would tilt the aft camera up instead of down. Cameras sit
+       at the mast origin (zero offset), so their positions are unchanged; only
+       orientation rotates. Roll component is unmeasured (needs port/stbd
+       horizon data); refine after the on-water test. See
+       docs/logs/2026/2026-07-20_gabby_logs.md. -->
+  <xacro:property name="cam_mast_pitch" value="${-1.85 * pi / 180.0}"/>
+  <link name="bizzy/camera_mast"/>
+  <joint name="base_to_camera_mast" type="fixed">
+    <parent link="bizzy/base_link"/>
+    <child link="bizzy/camera_mast"/>
+    <origin xyz="${cam_x} 0 ${cam_z}" rpy="0 ${cam_mast_pitch} 0"/>
+  </joint>
+  <xacro:oak_camera parent="bizzy/camera_mast" name="oak_forward"
+    x="0" y="0" z="0"
     pitch="${cam_tilt}" yaw="0"/>
-  <xacro:oak_camera parent="bizzy/base_link" name="oak_port"
-    x="${cam_x}" y="0" z="${cam_z}"
+  <xacro:oak_camera parent="bizzy/camera_mast" name="oak_port"
+    x="0" y="0" z="0"
     pitch="${cam_tilt}" yaw="${pi/2}"/>
-  <xacro:oak_camera parent="bizzy/base_link" name="oak_starboard"
-    x="${cam_x}" y="0" z="${cam_z}"
+  <xacro:oak_camera parent="bizzy/camera_mast" name="oak_starboard"
+    x="0" y="0" z="0"
     pitch="${cam_tilt}" yaw="${-pi/2}"/>
-  <xacro:oak_camera parent="bizzy/base_link" name="oak_aft"
-    x="${cam_x}" y="0" z="${cam_z}"
+  <xacro:oak_camera parent="bizzy/camera_mast" name="oak_aft"
+    x="0" y="0" z="0"
     pitch="${cam_tilt}" yaw="${pi}"/>
   <!-- ========== FCU GNSS Antennas (2x CUAV C-RTK 2HP) ========== -->

Commit message: fix(urdf): refine camera-mast calibration from 2026-07-20 recording
Calibrated against 1.43M waterline observations from the post-correction
bag (bag_2026-07-20T13.45.16_ffmpeg_seg), absolute-anchored by ray-casting
to the real Lake Massabesic shoreline (OSM) from the GNSS track:

- mast pitch: -1.85 -> -1.963 deg
- mast roll (previously unmeasured): +0.947 deg
- per-camera pitch/roll trims (bracket is not rigid: +-0.24 deg twist,
  aft camera in-view roll -1.7 deg)
- the field fix's +0.47 deg common-mode residual was finite-shore-distance
  geometry (atan(h/R)), not miscalibration; true common mode +0.01 deg
- properties renamed cam_* -> camera_* (no abbreviations)

Applying these values closes residuals on the same data to <=0.010 deg.
Method and reproduction scripts: docs/analysis/2026-07-20/README.md
(follow-up commit).

Refs #380

Co-Authored-By: Claude Fable 5 <noreply@anthropic.com>
Claude-Session: https://claude.ai/code/session_01Tukt1e7EaPzJvX96jWQp7G

File: bizzyboat_project11/urdf/bizzyboat.urdf.xacro (robot description, xacro)
@@ -131,7 +131,7 @@
        All tilted ~5deg downward (pitch = +0.09 rad in URDF convention).
        Positions are estimated [EST] — refine with measurements. -->
-  <xacro:property name="cam_x" value="0.31"/>
-  <xacro:property name="cam_z" value="1.41"/>
-  <xacro:property name="cam_tilt" value="0.09"/>
+  <xacro:property name="camera_x" value="0.31"/>
+  <xacro:property name="camera_z" value="1.41"/>
+  <xacro:property name="camera_tilt" value="0.09"/>
   <!-- Camera-mast remount correction (2026-07-20): a new mast brace left the
        whole 4-camera bracket pitched slightly bow-up, so the forward camera
@@ -142,29 +142,53 @@
        Modeled as ONE rotation of a common mast frame about base_link Y
        (bow-up = negative URDF pitch, opposite the +0.09 down-tilt), so all
-       four cameras rotate rigidly together. A per-camera cam_tilt change would
+       four cameras rotate rigidly together. A per-camera camera_tilt change would
        be wrong: it would tilt the aft camera up instead of down. Cameras sit
        at the mast origin (zero offset), so their positions are unchanged; only
-       orientation rotates. Roll component is unmeasured (needs port/stbd
-       horizon data); refine after the on-water test. See
-       docs/logs/2026/2026-07-20_gabby_logs.md. -->
-  <xacro:property name="cam_mast_pitch" value="${-1.85 * pi / 180.0}"/>
+       orientation rotates. See docs/logs/2026/2026-07-20_gabby_logs.md. -->
+  <!-- Refinement (2026-07-22, issue #380): calibrated against the 10-min
+       post-correction recording bag_2026-07-20T13.45.16_ffmpeg_seg — 1.43M
+       waterline observations (all 4 cameras, ~3000 frames each), absolute
+       reference = ray-cast to the real Lake Massabesic shoreline (OSM) from
+       the GNSS track. Two independent solves agree to <=0.08 deg; applying
+       these values closes residuals to <=0.011 deg on the same data.
+       Findings: field pitch -1.85 refined to -1.963 deg; roll (unmeasured in
+       the field) is +0.947 deg; the field's +0.47 deg common-mode residual
+       was finite-shore-distance geometry (atan(h/R)), not miscalibration.
+       The bracket is NOT perfectly rigid: per-camera trims below (pitch
+       relative to camera_tilt, roll about each camera's own axis) absorb a
+       +-0.24 deg twist mode and per-camera mount roll, largest on the aft
+       camera. Yaw trims are unobservable from waterline elevation and stay
+       at the cardinal directions. Uncertainty ~+-0.1 deg (systematic).
+       Method, data provenance, and reproduction scripts:
+       docs/analysis/2026-07-20/README.md -->
+  <xacro:property name="camera_mast_pitch" value="${-1.963 * pi / 180.0}"/>
+  <xacro:property name="camera_mast_roll" value="${0.947 * pi / 180.0}"/>
+  <!-- Per-camera trims (deg), same calibration:      pitch    roll -->
+  <xacro:property name="camera_trim_forward_pitch"  value="${ 0.107 * pi / 180.0}"/>
+  <xacro:property name="camera_trim_forward_roll"   value="${-0.572 * pi / 180.0}"/>
+  <xacro:property name="camera_trim_aft_pitch"  value="${ 0.467 * pi / 180.0}"/>
+  <xacro:property name="camera_trim_aft_roll"   value="${-0.777 * pi / 180.0}"/>
+  <xacro:property name="camera_trim_port_pitch" value="${-0.157 * pi / 180.0}"/>
+  <xacro:property name="camera_trim_port_roll"  value="${-0.031 * pi / 180.0}"/>
+  <xacro:property name="camera_trim_starboard_pitch" value="${-0.348 * pi / 180.0}"/>
+  <xacro:property name="camera_trim_starboard_roll"  value="${-0.385 * pi / 180.0}"/>
   <link name="bizzy/camera_mast"/>
   <joint name="base_to_camera_mast" type="fixed">
     <parent link="bizzy/base_link"/>
     <child link="bizzy/camera_mast"/>
-    <origin xyz="${cam_x} 0 ${cam_z}" rpy="0 ${cam_mast_pitch} 0"/>
+    <origin xyz="${camera_x} 0 ${camera_z}" rpy="${camera_mast_roll} ${camera_mast_pitch} 0"/>
   </joint>
   <xacro:oak_camera parent="bizzy/camera_mast" name="oak_forward"
     x="0" y="0" z="0"
-    pitch="${cam_tilt}" yaw="0"/>
+    roll="${camera_trim_forward_roll}" pitch="${camera_tilt + camera_trim_forward_pitch}" yaw="0"/>
   <xacro:oak_camera parent="bizzy/camera_mast" name="oak_port"
     x="0" y="0" z="0"
-    pitch="${cam_tilt}" yaw="${pi/2}"/>
+    roll="${camera_trim_port_roll}" pitch="${camera_tilt + camera_trim_port_pitch}" yaw="${pi/2}"/>
   <xacro:oak_camera parent="bizzy/camera_mast" name="oak_starboard"
     x="0" y="0" z="0"
-    pitch="${cam_tilt}" yaw="${-pi/2}"/>
+    roll="${camera_trim_starboard_roll}" pitch="${camera_tilt + camera_trim_starboard_pitch}" yaw="${-pi/2}"/>
   <xacro:oak_camera parent="bizzy/camera_mast" name="oak_aft"
     x="0" y="0" z="0"
-    pitch="${cam_tilt}" yaw="${pi}"/>
+    roll="${camera_trim_aft_roll}" pitch="${camera_tilt + camera_trim_aft_pitch}" yaw="${pi}"/>
   <!-- ========== FCU GNSS Antennas (2x CUAV C-RTK 2HP) ========== -->
   <!-- Black pucks fore and aft, feeding the Cube Orange FCU (moving-baseline
