Commit message: urdf: align sidescan channel joints with sibling macro style (#237)
Use pi math (${pi}/${-pi/2}/${pi/2}) and parent/child/origin element
ordering to match camera_oak/sonar macros. Rotations are identical
(pi == radians(180), etc.); frames unchanged. Addresses Copilot review on PR #238.

File: bizzyboat_project11/urdf/sensors/sidescan.xacro (robot description, xacro)
@@ -25,21 +25,21 @@
     <link name="bizzy/${name}_down"/>
     <joint name="${name}_to_${name}_down" type="fixed">
-      <origin xyz="0 0 0" rpy="${radians(180)} 0 0"/>
       <parent link="bizzy/${name}"/>
       <child link="bizzy/${name}_down"/>
+      <origin xyz="0 0 0" rpy="${pi} 0 0"/>
     </joint>
     <!-- Port side-scan beam: +Z to port (+Y). -->
     <link name="bizzy/${name}_port"/>
     <joint name="${name}_to_${name}_port" type="fixed">
-      <origin xyz="0 0 0" rpy="${radians(-90)} 0 0"/>
       <parent link="bizzy/${name}"/>
       <child link="bizzy/${name}_port"/>
+      <origin xyz="0 0 0" rpy="${-pi/2} 0 0"/>
     </joint>
     <!-- Starboard side-scan beam: +Z to starboard (-Y). -->
     <link name="bizzy/${name}_starboard"/>
     <joint name="${name}_to_${name}_starboard" type="fixed">
-      <origin xyz="0 0 0" rpy="${radians(90)} 0 0"/>
       <parent link="bizzy/${name}"/>
       <child link="bizzy/${name}_starboard"/>
+      <origin xyz="0 0 0" rpy="${pi/2} 0 0"/>
     </joint>
   </xacro:macro>

Commit message: fix(bizzyboat): sidescan grazing_deg default 62.5° → 35° (field-measured)
The 62.5° half-fan-off-nadir default from #303 was a tiling heuristic ~27°
too steep. Offline analysis of field sonar bags (Massabesic + bizzy runs)
puts the SideVü boresight depression at ~35°: the bottom-return angular
profile I(φ)=asin(nadir_depth/slant_range) peaks ~38°, less a few degrees
of near-nadir backscatter steep-bias. A roll-day regression (steep-edge vs
vessel roll, opposite-sign ±1 slopes per channel) validated the geometry,
and it matches the recreational side-imaging patent norm (~20-40°, nom 30°).
Rationale comment rewritten; grazing_deg stays overridable.

Closes #305. Part of #185.

File: bizzyboat_project11/urdf/sensors/sidescan.xacro (robot description, xacro)
@@ -15,14 +15,21 @@
        while +X stays forward — marine_sidescan_mosaic (#200) extracts heading
        from +Z via ecefPoseToGeoBeam and consumes exactly this tilted boresight.
-       Default grazing_deg = 62.5 = 90 - SideVu_fan/2 = 90 - 27.5 (half the
-       55-deg SideVu fan off nadir). This places the INNER edge of the fan at
-       nadir, tiling cleanly against the _down (ClearVu) beam with no nadir gap
-       or overlap. The fan half-width (55 deg) is published by the driver per
-       marine_tools#62, so this default can be refined after calibration.
-       Alternative: classic side-imaging aims the boresight ~20-30 deg below
-       horizontal for longer far across-track range; set grazing_deg to that
-       after field calibration if desired (it trades the clean nadir tiling for
-       a nadir gap). The default keeps the nadir seam clean out of the box. -->
-  <xacro:macro name="garmin_sidescan" params="parent name x:=0 y:=0 z:=0 grazing_deg:=62.5">
+       Default grazing_deg = 35 (boresight depression below horizontal),
+       MEASURED from field sonar bags (Massabesic + bizzy runs, 2026-06-21):
+       the bottom-return angular profile I(phi) = asin(nadir_depth / slant_range)
+       peaks near 38 deg, and the near-nadir backscatter steep-bias puts the true
+       boresight a few degrees shallower (~35). A roll-day regression (per-ping
+       steep-edge vs vessel roll, opposite-sign +/-1 slopes per channel)
+       validated the geometry. This matches the recreational side-imaging norm
+       of ~20-40 deg, nominal ~30 (Garmin/Humminbird/Navico patents:
+       US7652952B2, US11137495B2); survey towfish run ~10.
+       This is NOT the 90 - fan/2 = 62.5 "half-fan off nadir" that once shipped
+       (#303) — that was a tiling heuristic, ~27 deg too steep, and not how a
+       side-imaging sonar is aimed. The 55-deg fan (published by the driver,
+       marine_tools#62) could not be cleanly cross-checked here (the shallow
+       -3 dB edge falls outside the range window in shallow water; a 50-60 m
+       range pass over 10-15 m water would resolve it). Override grazing_deg
+       for further calibration. See issue #305 / #185. -->
+  <xacro:macro name="garmin_sidescan" params="parent name x:=0 y:=0 z:=0 grazing_deg:=35.0">
     <!-- Mount frame, aligned with base_link (X fwd, Y port, Z up). -->
     <link name="bizzy/${name}"/>
